File: KiCAD/biron.kicad_pcb (KiCad board)
At the start: 4 copper layers, 162.6 x 100.3 mm, 141 parts, among them J5 USB_B_Mini, J6 USB_B_Mini, J9 Molex KK-254, Q1 DMN15H310SK3-13, Q2 DMN15H310SK3-13, Q3 DMN15H310SK3-13, Q4 IPP50R140CPXKSA1, Q5 IPP50R140CPXKSA1, Q6 2N7002, Q7 2N7002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

Commit message: Update Text
Other:
- board text added: "A"
- board text added: "B"
- board text added: "BATT+"
- board text added: "BATT-"
- board text added: "K-Type"
- board text added: "LittelFuse Mini 897 10A"
- board text added: "OUT1"
- board text added: "OUT2"
Changed lines of the file:
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@@
     (property "Sheetname" "")
     (attr through_hole)
-    (fp_text reference "J2" (at -4.445 0 unlocked) (layer "F.SilkS")
+    (fp_text reference "J2" (at -1.27 -3.175 unlocked) (layer "F.SilkS")
         (effects (font (size 1 1) (thickness 0.1)))
     )
@@
     (property "Sheetname" "")
     (attr through_hole)
-    (fp_text reference "J1" (at -4.445 0 unlocked) (layer "F.SilkS")
+    (fp_text reference "J1" (at -1.905 -3.175 unlocked) (layer "F.SilkS")
         (effects (font (size 1 1) (thickness 0.1)))
     )
@@
     (property "ki_keywords" "fuse")
     (attr through_hole)
-    (fp_text reference "F1" (at -11.815 -0.205) (layer "F.SilkS")
+    (fp_text reference "F1" (at -9.14 -4.24) (layer "F.SilkS")
         (effects (font (size 1 1) (thickness 0.15)))
     )
@@
     (effects (font (size 1 1) (thickness 0.15) italic) (justify left bottom mirror))
   )
+  (gr_text "BATT+" (at 62.865 95.885) (layer "F.SilkS")
+    (effects (font (size 1 1) (thickness 0.15)) (justify left bottom))
+  )
+  (gr_text "OUT2" (at 55.245 145.415) (layer "F.SilkS")
+    (effects (font (size 1.5 1.5) (thickness 0.3) bold))
+  )
+  (gr_text "A" (at 193.675 132.715) (layer "F.SilkS")
+    (effects (font (size 1.5 1.5) (thickness 0.3) bold))
+  )
   (gr_text "USB" (at 149.86 64.77 90) (layer "F.SilkS")
     (effects (font (size 1.5 1.5) (thickness 0.3) bold) (justify left bottom))
   )
+  (gr_text "BATT-" (at 62.865 88.9) (layer "F.SilkS")
+    (effects (font (size 1 1) (thickness 0.15)) (justify left bottom))
+  )
+  (gr_text "OUT1" (at 54.61 119.38) (layer "F.SilkS")
+    (effects (font (size 1.5 1.5) (thickness 0.3) bold))
+  )
   (gr_text "UART" (at 130.81 64.77 90) (layer "F.SilkS")
     (effects (font (size 1.5 1.5) (thickness 0.3) bold) (justify left bottom))
   )
+  (gr_text "LittelFuse Mini 897 10A" (at 48.26 112.395) (layer "F.SilkS")
+    (effects (font (size 1.5 1.5) (thickness 0.3) bold) (justify left bottom))
+  )
   (gr_text "120R" (at 117.475 65.405 90) (layer "F.SilkS")
     (effects (font (size 1 1) (thickness 0.15)) (justify bottom))
   )
+  (gr_text "B" (at 193.675 118.11) (layer "F.SilkS")
+    (effects (font (size 1.5 1.5) (thickness 0.3) bold))
+  )
+  (gr_text "K-Type" (at 199.39 111.125) (layer "F.SilkS")
+    (effects (font (size 2 2) (thickness 0.4) bold))
+  )
   (segment (start 187.345 126.365) (end 191.77 126.365) (width 0.508) (layer "F.Cu") (net 1))

Commit message: Update PCB silkscreen
Other:
- board text added: "BOOT"
- board text added: "RST"
